Commit message: Added visualization

File: robots/flexiv/robot.urdf (robot description, URDF)
Before this commit: robot flexivArm, 9 links, 8 joints
Links:
- link link1: mass 3.626054 -> 3.463530
- link link2: mass 2.686237 -> 2.461088
- link link3: mass 2.266909 -> 2.114110
- link link4: mass 2.266909 -> 2.114110
- link link5: mass 2.168938 -> 2.007245
- link link6: mass 2.037469 -> 1.953128
- link link7: mass 0.878548 -> 0.789282
Joints:
- joint joint1: limit lower=-2.87979 upper=2.87979 effort=90 velocity=2.61799 -> lower=-2.87979 upper=2.87979 effort=123 velocity=2.61799
- joint joint2: limit lower=-2.16421 upper=2.16421 effort=90 velocity=2.61799 -> lower=-2.16421 upper=2.16421 effort=123 velocity=2.61799
- joint joint3: limit lower=-3.05433 upper=3.05433 effort=40 velocity=2.61799 -> lower=-3.05433 upper=3.05433 effort=64 velocity=2.61799
- joint joint4: axis 0 1 0 -> 0 -1 0; limit lower=-2.79253 upper=1.95477 effort=40 velocity=2.61799 -> lower=-2.79253 upper=1.95477 effort=64 velocity=2.61799
- joint joint5: limit lower=-3.05433 upper=3.05433 effort=20 velocity=5.23599 -> lower=-3.05433 upper=3.05433 effort=39 velocity=5.23599
- joint joint6: limit lower=-1.48353 upper=4.62512 effort=20 velocity=5.23599 -> lower=-1.48353 upper=4.62512 effort=39 velocity=5.23599
- joint joint7: limit lower=-3.05433 upper=3.05433 effort=20 velocity=5.23599 -> lower=-3.05433 upper=3.05433 effort=39 velocity=5.23599
